File: Feather-ZED-F9P-GPS.kicad_pcb (KiCad board)
At the start: 2 copper layers, 61 x 59 mm, 69 parts, among them J1 Conn_01x12, J2 Conn_01x16, J3 USB_B_Micro, J4 Conn_01x7, J5 Conn_01x05, J7 Conn_01x06, U1 ZED-F9P, U2 AP2112K-3.3

Commit message: Some edits?
Some edits I made a while ago apparently? Don't remember the details but I'll push anways
Parts:
- removed J4: Conn_01x7, Connector_PinSocket_2.54mm:PinSocket_1x07_P2.54mm_Vertical
- removed J5: Conn_01x05, Connector_PinSocket_2.54mm:PinSocket_1x05_P2.54mm_Vertical
- removed J7: Conn_01x06, Connector_PinSocket_2.54mm:PinSocket_1x06_P2.54mm_Vertical
- removed JP6: Cut to remove I2C Pullups, Jumper:SolderJumper-2_P1.3mm_Bridged_RoundedPad1.0x1.5mm
- removed ~CS1: ~CS, Connector_Pin:Pin_D1.0mm_L10.0mm
- added D8: BAT60AE6327HTSA1, SamacSys_Parts:SOD2513X110N, F.Cu at (125.3, 33.1)
- added D9: BAT60AE6327HTSA1, SamacSys_Parts:SOD2513X110N, F.Cu at (43.1, 105.2)
- C1, C2, C3, C4, C5, C6, C7, C8: footprint Capacitor_SMD:C_0805_2012Metric -> Capacitor_SMD:C_0603_1608Metric
- JP4: value Cut to remove I2C Pullups -> SolderJumper_3_Bridged123; footprint Jumper:SolderJumper-2_P1.3mm_Bridged_RoundedPad1.0x1.5mm -> SamacSys_Parts:SMT-JUMPER_3_2-NC_TRACE_SILK
- L1: footprint Inductor_SMD:L_0805_2012Metric -> Inductor_SMD:L_0603_1608Metric
- R1, R2, R5: footprint Resistor_SMD:R_0805_2012Metric -> Resistor_SMD:R_0603_1608Metric
- R10, R11, R12, R13, R14, R15, R16, R17, R18, R19, R20, R21, R22, R23, R3, R4, R6, R7, R8, R9: footprint Capacitor_SMD:C_0805_2012Metric -> Resistor_SMD:R_0603_1608Metric
- U.FL: renamed from AE1; value Antenna_Chip -> U.FL
- moved BT1 58.7 mm to (19.7, 91.7)
- moved C7 58.4 mm to (130.0, 33.9)
- moved C4 58.4 mm to (128.9, 49.6)
- moved C5 58.4 mm to (131.0, 42.8)
- moved C6 58.4 mm to (129.3, 29.3)
- moved C8 58.4 mm to (130.6, 32.0)
- moved D6 58.4 mm to (131.4, 25.8)
- moved R10 58.4 mm to (120.0, 22.8)
- moved R3 58.4 mm to (120.7, 30.5)
- moved R4 58.4 mm to (123.3, 30.3)
- moved R5 58.4 mm to (130.9, 49.8)
- moved C2 58.4 mm to (130.0, 39.1)
- moved C3 58.4 mm to (130.0, 40.9)
- moved D1 58.4 mm to (131.7, 46.5)
- moved IC1 58.4 mm to (127.4, 25.1)
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Connections:
- C7 pad 1: +3V3 -> Net-(C7-Pad1)
- C8 pad 1: +3V3 -> Net-(C7-Pad1)
- J2 pad 2: +3V3 -> Net-(D9-Pad2)
- JP4 pad 1: +3V3 -> Net-(JP4-Pad1)
- JP4 pad 2: Net-(JP4-Pad2) -> +3V3
- R22 pad 2: Net-(JP4-Pad2) -> Net-(JP4-Pad3)
- R23 pad 2: Net-(JP6-Pad2) -> Net-(JP4-Pad1)
- U2 pad 5: +3V3 -> Net-(C7-Pad1)
Routing:
- net /SCL-SCK: track 126.7 -> 0.00 mm, vias 2 -> 0
- net +3V3: track 122.9 -> 0.00 mm, vias 1 -> 0
- net /RXI-MOSI: track 118.1 -> 0.00 mm, vias 4 -> 0
- net /TX0-MISO: track 116.5 -> 0.00 mm, vias 4 -> 0
- net /SDA-~CS: track 110.9 -> 0.00 mm, vias 1 -> 0
- net GND: track 105.8 -> 0.00 mm, vias 366 -> 59
- net /TX2: track 79.9 -> 0.00 mm, vias 2 -> 0
- net /RX2: track 77.8 -> 0.00 mm, vias 2 -> 0
- net /PPS: track 68.1 -> 0.00 mm, vias 2 -> 0
- net /SDA: track 45.3 -> 0.00 mm, vias 1 -> 0
- net +5V: track 37.7 -> 0.00 mm
- net /FENCE_STAT: track 36.1 -> 0.00 mm, vias 2 -> 0
- net /12: track 36.0 -> 0.00 mm
- net /RTK_STAT: track 34.1 -> 0.00 mm, vias 2 -> 0
- net /SCL: track 33.8 -> 0.00 mm, vias 1 -> 0
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Other:
- board size 61 x 59 mm -> 50.8 x 22.9 mm
- board text removed: "+3V"
- board text removed: "+5V"
- board text removed: "12 11 10 9 6 5"
- board text removed: "5 6 9 10 11 12"
- board text removed: "Available ~CS~ Pins"
- board text removed: "GND"
- board text removed: "I2C Pullups"
- board text removed: "INT"
- board text removed: "RX2"
- board text removed: "TX2"
- board text removed: "~RESET"
- board text removed: "~SAFE"
