File: Feather-ZED-F9P-GPS.sch (KiCad schematic (older format))
At the start: 65 parts, among them J1 Conn_01x12, J2 Conn_01x16, J3 USB_B_Micro, J4 Conn_01x7, J5 Conn_01x05, J7 Conn_01x06, U1 ZED-F9P, U2 AP2112K-3.3

Commit message: Some edits?
Some edits I made a while ago apparently? Don't remember the details but I'll push anways
Parts:
- removed JP4, JP6: Cut to remove I2C Pullups, Jumper:SolderJumper-2_P1.3mm_Bridged_RoundedPad1.0x1.5mm, symbol Jumper:SolderJumper_2_Bridged
- added D8, D9: BAT60AE6327HTSA1, SOD2513X110N, symbol Device:D
- added JP4: SolderJumper_3_Bridged123, SamacSys_Parts:SMT-JUMPER_3_2-NC_TRACE_SILK, symbol Jumper:SolderJumper_3_Bridged123
- AE1: value Antenna_Chip -> U.FL
- C1, C2, C3, C4, C5, C6, C7, C8: footprint Capacitor_SMD:C_0805_2012Metric -> Capacitor_SMD:C_0603_1608Metric
- J4: footprint Connector_PinSocket_2.54mm:PinSocket_1x07_P2.54mm_Vertical -> ~Connector_PinSocket_2.54mm:PinSocket_1x07_P2.54mm_Vertical
- J5: footprint Connector_PinSocket_2.54mm:PinSocket_1x05_P2.54mm_Vertical -> ~Connector_PinSocket_2.54mm:PinSocket_1x05_P2.54mm_Vertical
- J7: footprint Connector_PinSocket_2.54mm:PinSocket_1x06_P2.54mm_Vertical -> ~Connector_PinSocket_2.54mm:PinSocket_1x06_P2.54mm_Vertical
- L1: footprint Inductor_SMD:L_0805_2012Metric -> Inductor_SMD:L_0603_1608Metric
- R1, R2, R5: footprint Resistor_SMD:R_0805_2012Metric -> Resistor_SMD:R_0603_1608Metric
- R10, R11, R12, R13, R14, R15, R16, R17, R18, R19, R20, R21, R22, R23, R3, R4, R6, R7, R8, R9: footprint Capacitor_SMD:C_0805_2012Metric -> Resistor_SMD:R_0603_1608Metric
- ~CS1: footprint Connector_Pin:Pin_D1.0mm_L10.0mm -> ~Connector_Pin:Pin_D1.0mm_L10.0mm
Connections:
- net +3V3: now also D8.1 (K), D9.1 (K), JP4.2 (C); no longer C7.1, C8.1, J2.2 (Pin_2), U2.5 (VOUT)
- net at R22.2: now also JP4.3 (B)
- net at R23.2: now also JP4.1 (A)
- new net: D9.2 (A), J2.2 (Pin_2)
- new net: C7.1, C8.1, D8.2 (A), U2.5 (VOUT)
Other:
- moved on the sheet: J4, J5, J7, ~{CS1}
